Commit message: feat: moving a 4 wheels vehicule

File: ackerman_robot/model/example.xacro (robot description, xacro)
@@ -85,5 +85,5 @@
         </collision>
         <inertial>
-            <mass value="0.5"/>
+            <mass value="0.01"/>
             <inertia ixx="0.01" ixy="0" ixz="0" iyy="0.01" iyz="0" izz="0.01"/>
         </inertial>
@@ -103,5 +103,5 @@
         </collision>
         <inertial>
-            <mass value="0.5"/>
+            <mass value="0.01"/>
             <inertia ixx="0.01" ixy="0" ixz="0" iyy="0.01" iyz="0" izz="0.01"/>
         </inertial>
@@ -175,4 +175,14 @@
     </gazebo>
     <gazebo reference="caster_wheel">
+        <material>Gazebo/Black</material>
+        <mu1 value="0.1"/>
+        <mu2 value="0.1"/>
+    </gazebo>
+    <gazebo reference="back_right_wheel">
+        <material>Gazebo/Black</material>
+        <mu1 value="1.0"/>
+        <mu2 value="1.0"/>
+    </gazebo>
+    <gazebo reference="back_left_wheel">
         <material>Gazebo/Black</material>
         <mu1 value="0.1"/>
