Commit message: fix(ackerman_robot): send message for brushless

File: ackerman_robot/urdf/ackermann.urdf.xacro (robot description, xacro)
@@ -156,5 +156,5 @@
         <inertial>
             <mass value="11.3" />
-             <inertia ixx="0.026" ixy="0.0" ixz="0.0" iyy="0.026" iyz="0.0" izz="0.051" />
+             <inertia ixx="0.026" ixy="0.0" ixz="0.0" iyy="0.026" iyz="0.0" izz="0.051"/>
         </inertial>
     </link>

Commit message: feat(ackerman_robot): put bycicle_controller working

File: ackerman_robot/urdf/ackermann.urdf.xacro (robot description, xacro)
@@ -167,5 +167,5 @@
     </joint>
     <ros2_control name="OnyCroit" type="system">
-      <hardware>
+      <!--<hardware>
         <plugin>ackerman_robot/DiffDriveArduinoHardware</plugin>
         <param name="front_left_wheel_name">left_wheel_steering_joint</param>
@@ -200,4 +200,27 @@
         <command_interface name="position" />
         <state_interface name="position" />
+        </joint>-->
+        <hardware>
+            <plugin>ackerman_robot/DiffDriveArduinoHardware</plugin>
+            <param name="example_param_hw_start_duration_sec">0</param>
+            <param name="example_param_hw_stop_duration_sec">3.0</param>
+               <param name="loop_rate">30</param>
+        <param name="device">/dev/ttyACM0</param>
+        <param name="baud_rate">9600</param>
+        <param name="timeout_ms">1000</param>
+        <param name="enc_counts_per_rev">3436</param>
+        <param name="pid_p">20</param>
+        <param name="pid_d">12</param>
+        <param name="pid_i">0</param>
+        <param name="pid_o">50</param>
+        </hardware>
+        <joint name="left_wheel_steering_joint">
+            <command_interface name="position"/>
+            <state_interface name="position"/>
+        </joint>
+        <joint name="rear_left_wheel_joint">
+            <command_interface name="velocity"/>
+            <state_interface name="velocity"/>
+            <state_interface name="position"/>
         </joint>
     </ros2_control>

Commit message: ackerman_robot: fixed delay between hardware interface and hardware

File: ackerman_robot/urdf/ackermann.urdf.xacro (robot description, xacro)
@@ -167,5 +167,5 @@
     </joint>
     <ros2_control name="OnyCroit" type="system">
-      <!--<hardware>
+      <hardware>
         <plugin>ackerman_robot/DiffDriveArduinoHardware</plugin>
         <param name="front_left_wheel_name">left_wheel_steering_joint</param>
@@ -175,5 +175,5 @@
         <param name="loop_rate">30</param>
         <param name="device">/dev/ttyACM0</param>
-        <param name="baud_rate">9600</param>
+        <param name="baud_rate">115200</param>
         <param name="timeout_ms">1000</param>
         <param name="enc_counts_per_rev">3436</param>
@@ -200,6 +200,6 @@
         <command_interface name="position" />
         <state_interface name="position" />
-        </joint>-->
-        <hardware>
+        </joint>
+        <!--<hardware>
             <plugin>ackerman_robot/DiffDriveArduinoHardware</plugin>
             <param name="example_param_hw_start_duration_sec">0</param>
@@ -223,5 +223,5 @@
             <state_interface name="velocity"/>
             <state_interface name="position"/>
-        </joint>
+        </joint>-->
     </ros2_control>
   <!--  <ros2_control name="GazeboSystem" type="system">

Commit message: feat: updated documentation for hardware

File: ackerman_robot/urdf/ackermann.urdf.xacro (robot description, xacro)
@@ -201,27 +201,4 @@
         <state_interface name="position" />
         </joint>
-        <!--<hardware>
-            <plugin>ackerman_robot/DiffDriveArduinoHardware</plugin>
-            <param name="example_param_hw_start_duration_sec">0</param>
-            <param name="example_param_hw_stop_duration_sec">3.0</param>
-               <param name="loop_rate">30</param>
-        <param name="device">/dev/ttyACM0</param>
-        <param name="baud_rate">9600</param>
-        <param name="timeout_ms">1000</param>
-        <param name="enc_counts_per_rev">3436</param>
-        <param name="pid_p">20</param>
-        <param name="pid_d">12</param>
-        <param name="pid_i">0</param>
-        <param name="pid_o">50</param>
-        </hardware>
-        <joint name="left_wheel_steering_joint">
-            <command_interface name="position"/>
-            <state_interface name="position"/>
-        </joint>
-        <joint name="rear_left_wheel_joint">
-            <command_interface name="velocity"/>
-            <state_interface name="velocity"/>
-            <state_interface name="position"/>
-        </joint>-->
     </ros2_control>
   <!--  <ros2_control name="GazeboSystem" type="system">
@@ -250,5 +227,5 @@
     <!--<gazebo>
         <plugin filename="gz_ros2_control-system" name="gz_ros2_control::GazeboSimROS2ControlPlugin">
-            <parameters>$(find ackerman_robot)/config/ackermann_drive_controller.yaml</parameters>
+            <parameters>$(find ackerman_robot)/config/ackermann_controller.yaml</parameters>
         </plugin>
     </gazebo>-->

Commit message: enabling using hardware and gazebo

File: ackerman_robot/urdf/ackermann.urdf.xacro (robot description, xacro)
@@ -13,4 +13,5 @@
         <color rgba="1 1 1 1" />
     </material>
+    <xacro:arg name="sim_mode" default="false"/>
     <link name="base_link" />
     <!-- Chassis -->
@@ -166,26 +167,52 @@
         <dynamics damping="0.2" />
     </joint>
-    <ros2_control name="OnyCroit" type="system">
-      <hardware>
-        <plugin>ackerman_robot/DiffDriveArduinoHardware</plugin>
-        <param name="front_left_wheel_name">left_wheel_steering_joint</param>
-        <param name="front_right_wheel_name">right_wheel_steering_joint</param>
-        <param name="rear_left_wheel_name">rear_left_wheel_joint</param>
-        <param name="rear_right_wheel_name">rear_right_wheel_joint</param>
-        <param name="loop_rate">30</param>
-        <param name="device">/dev/ttyACM0</param>
-        <param name="baud_rate">115200</param>
-        <param name="timeout_ms">1000</param>
-        <param name="enc_counts_per_rev">3436</param>
-        <param name="pid_p">20</param>
-        <param name="pid_d">12</param>
-        <param name="pid_i">0</param>
-        <param name="pid_o">50</param>
-      </hardware>
-      <joint name="rear_left_wheel_joint">
-      <command_interface name="velocity" />
-      <state_interface name="velocity" />
-      <state_interface name="position" />
-      </joint>
+    <xacro:unless value="$(arg sim_mode)">
+        <ros2_control name="OnyCroit" type="system">
+        <hardware>
+            <plugin>ackerman_robot/DiffDriveArduinoHardware</plugin>
+            <param name="front_left_wheel_name">left_wheel_steering_joint</param>
+            <param name="front_right_wheel_name">right_wheel_steering_joint</param>
+            <param name="rear_left_wheel_name">rear_left_wheel_joint</param>
+            <param name="rear_right_wheel_name">rear_right_wheel_joint</param>
+            <param name="loop_rate">30</param>
+            <param name="device">/dev/ttyACM0</param>
+            <param name="baud_rate">115200</param>
+            <param name="timeout_ms">1000</param>
+            <param name="enc_counts_per_rev">3436</param>
+            <param name="pid_p">20</param>
+            <param name="pid_d">12</param>
+            <param name="pid_i">0</param>
+            <param name="pid_o">50</param>
+        </hardware>
+        <joint name="rear_left_wheel_joint">
+        <command_interface name="velocity" />
+        <state_interface name="velocity" />
+        <state_interface name="position" />
+        </joint>
+            <joint name="rear_right_wheel_joint">
+            <command_interface name="velocity" />
+            <state_interface name="velocity" />
+            <state_interface name="position" />
+            </joint>
+            <joint name="left_wheel_steering_joint">
+            <command_interface name="position" />
+            <state_interface name="position" />
+            </joint>
+            <joint name="right_wheel_steering_joint">
+            <command_interface name="position" />
+            <state_interface name="position" />
+            </joint>
+        </ros2_control>
+    </xacro:unless>
+  <xacro:if value="$(arg sim_mode)">
+    <ros2_control name="GazeboSystem" type="system">
+        <hardware>
+        <plugin>gz_ros2_control/GazeboSimSystem</plugin>
+        </hardware>
+        <joint name="rear_left_wheel_joint">
+        <command_interface name="velocity" />
+        <state_interface name="velocity" />
+        <state_interface name="position" />
+        </joint>
         <joint name="rear_right_wheel_joint">
         <command_interface name="velocity" />
@@ -202,31 +229,9 @@
         </joint>
     </ros2_control>
-  <!--  <ros2_control name="GazeboSystem" type="system">
-    <hardware>
-      <plugin>gz_ros2_control/GazeboSimSystem</plugin>
-    </hardware>
-    <joint name="rear_left_wheel_joint">
-      <command_interface name="velocity" />
-      <state_interface name="velocity" />
-      <state_interface name="position" />
-    </joint>
-    <joint name="rear_right_wheel_joint">
-      <command_interface name="velocity" />
-      <state_interface name="velocity" />
-      <state_interface name="position" />
-    </joint>
-    <joint name="left_wheel_steering_joint">
-      <command_interface name="position" />
-      <state_interface name="position" />
-    </joint>
-    <joint name="right_wheel_steering_joint">
-      <command_interface name="position" />
-      <state_interface name="position" />
-    </joint>
-  </ros2_control>-->
-    <!--<gazebo>
-        <plugin filename="gz_ros2_control-system" name="gz_ros2_control::GazeboSimROS2ControlPlugin">
-            <parameters>$(find ackerman_robot)/config/ackermann_controller.yaml</parameters>
-        </plugin>
-    </gazebo>-->
+        <gazebo>
+            <plugin filename="gz_ros2_control-system" name="gz_ros2_control::GazeboSimROS2ControlPlugin">
+                <parameters>$(find ackerman_robot)/config/ackermann_controller.yaml</parameters>
+            </plugin>
+        </gazebo>
+    </xacro:if>
 </robot>

Commit message: ackerman_robot: update xacro file lengths and widths

File: ackerman_robot/urdf/ackermann.urdf.xacro (robot description, xacro)
@@ -13,4 +13,13 @@
         <color rgba="1 1 1 1" />
     </material>
+    <!-- Define robot constants -->
+    <xacro:property name="base_width" value="0.117"/>
+    <xacro:property name="base_length" value="0.183"/>
+    <xacro:property name="base_height" value="0.05"/>
+    <xacro:property name="wheel_radius" value="0.03"/>
+    <xacro:property name="wheel_width" value="0.02"/>
+    <xacro:property name="wheel_ygap" value="0.025"/>
+    <xacro:property name="wheel_zoff" value="0.05"/>
+    <xacro:property name="wheel_xoff" value="0.12"/>
     <xacro:arg name="sim_mode" default="false"/>
     <link name="base_link" />
@@ -20,5 +29,5 @@
             <origin xyz="0 0 0" rpy="0 0 0" />
             <geometry>
-                <box size="0.183 0.117 0.05" />
+                <box size="${base_length} ${base_width} ${base_height}" />
             </geometry>
         </collision>
@@ -26,5 +35,5 @@
             <origin xyz="0 0 0" rpy="0 0 0" />
             <geometry>
-                <box size="0.183 0.117 0.05" />
+                <box size="${base_length} ${base_width} ${base_height}" />
             </geometry>
             <material name="Orange" />
@@ -70,10 +79,10 @@
         <collision>
             <geometry>
-                <cylinder length="0.02" radius="0.03" />
-            </geometry>
-        </collision>
-        <visual>
-            <geometry>
-                <cylinder length="0.02" radius="0.03" />
+                <cylinder length="${wheel_width}" radius="${wheel_radius}" />
+            </geometry>
+        </collision>
+        <visual>
+            <geometry>
+                <cylinder length="${wheel_width}" radius="${wheel_radius}" />
             </geometry>
             <material name="Black" />
@@ -122,10 +131,10 @@
         <collision>
             <geometry>
-                <cylinder length="0.03" radius="0.03" />
-            </geometry>
-        </collision>
-        <visual>
-            <geometry>
-                <cylinder length="0.03" radius="0.03" />
+                <cylinder length="${wheel_width}" radius="${wheel_radius}" />
+            </geometry>
+        </collision>
+        <visual>
+            <geometry>
+                <cylinder length="${wheel_width}" radius="${wheel_radius}" />
             </geometry>
             <material name="Black" />
@@ -146,10 +155,10 @@
         <collision>
             <geometry>
-                <cylinder length="0.02" radius="0.03" />
-            </geometry>
-        </collision>
-        <visual>
-            <geometry>
-                <cylinder length="0.02" radius="0.03" />
+                <cylinder length="${wheel_width}" radius="${wheel_radius}" />
+            </geometry>
+        </collision>
+        <visual>
+            <geometry>
+                <cylinder length="${wheel_width}" radius="${wheel_radius}"/>
             </geometry>
             <material name="Black" />

Commit message: ackerman_robot: updating values en .xacro

File: ackerman_robot/urdf/ackermann.urdf.xacro (robot description, xacro)
@@ -17,6 +17,8 @@
     <xacro:property name="base_length" value="0.183"/>
     <xacro:property name="base_height" value="0.05"/>
+    <xacro:property name="base_mass" value="120"/>
     <xacro:property name="wheel_radius" value="0.03"/>
     <xacro:property name="wheel_width" value="0.02"/>
+    <xacro:property name="wheel_mass" value="11"/>
     <xacro:property name="wheel_ygap" value="0.025"/>
     <xacro:property name="wheel_zoff" value="0.05"/>
@@ -41,6 +43,8 @@
         <inertial>
             <origin xyz="0 0 0" rpy="0 0 0" />
-            <mass value="100" />
-            <inertia ixx="1.04" ixy="0.0" ixz="0.0" iyy="3.54" iyz="0.0" izz="4.166" />
+            <mass value="${base_mass}" />
+            <inertia ixx="${1/12 * base_mass * (base_height**2 + base_length ** 2)}" ixy="0.0" ixz="0.0"
+            iyy="${1/12 * base_mass * (base_height ** 2 + base_width ** 2)}" iyz="0.0"
+            izz="${1/12 * base_mass * (base_width ** 2 + base_length ** 2)}" />
         </inertial>
     </link>
@@ -54,16 +58,18 @@
         <collision>
             <geometry>
-                <cylinder length="0.02" radius="0.03" />
-            </geometry>
-        </collision>
-        <visual>
-            <geometry>
-                <cylinder length="0.02" radius="0.03" />
-            </geometry>
-            <material name="Black" />
-        </visual>
-        <inertial>
-            <mass value="11.3" />
-            <inertia ixx="0.026" ixy="0.0" ixz="0.0" iyy="0.026" iyz="0.0" izz="0.051" />
+                <cylinder length="${wheel_width}" radius="${wheel_radius}" />
+            </geometry>
+        </collision>
+        <visual>
+            <geometry>
+                <cylinder length="${wheel_width}" radius="${wheel_radius}" />
+            </geometry>
+            <material name="Black" />
+        </visual>
+        <inertial>
+           <mass value="${base_mass}" />
+           <inertia ixx="${1/12 * base_mass * (base_height**2 + base_length ** 2)}" ixy="0.0" ixz="0.0"
+            iyy="${1/12 * base_mass * (base_height ** 2 + base_width ** 2)}" iyz="0.0"
+            izz="${1/12 * base_mass * (base_width ** 2 + base_length ** 2)}" />
         </inertial>
     </link>
@@ -89,6 +95,9 @@
         </visual>
         <inertial>
-            <mass value="11.3" />
-            <inertia ixx="0.026" ixy="0.0" ixz="0.0" iyy="0.026" iyz="0.0" izz="0.051" />
+            <mass value="${wheel_mass}" />
+            <inertia ixx="${1/12*wheel_mass*(3*wheel_radius**2+wheel_width)}"
+            ixy="0.0" ixz="0.0"
+            iyy="${1/12*wheel_mass*(3*wheel_radius**2+wheel_width)}"  iyz="0.0"
+            izz="${1/12*wheel_mass*wheel_radius**2}" />
         </inertial>
     </link>
@@ -116,6 +125,9 @@
     <link name="right_wheel_steering">
         <inertial>
-            <mass value="0.1"/>
-            <inertia ixx="0.26" ixy="0.0" ixz="0.0" iyy="0.26" iyz="0.0" izz="0.51" />
+           <mass value="${wheel_mass}" />
+            <inertia ixx="${1/12*wheel_mass*(3*wheel_radius**2+wheel_width)}"
+            ixy="0.0" ixz="0.0"
+            iyy="${1/12*wheel_mass*(3*wheel_radius**2+wheel_width)}"  iyz="0.0"
+            izz="${1/12*wheel_mass*wheel_radius**2}" />
         </inertial>
     </link>
@@ -141,6 +153,9 @@
         </visual>
         <inertial>
-            <mass value="11.3" />
-            <inertia ixx="0.26" ixy="0.0" ixz="0.0" iyy="0.26" iyz="0.0" izz="0.51" />
+            <mass value="${wheel_mass}" />
+            <inertia ixx="${1/12*wheel_mass*(3*wheel_radius**2+wheel_width)}"
+            ixy="0.0" ixz="0.0"
+            iyy="${1/12*wheel_mass*(3*wheel_radius**2+wheel_width)}"  iyz="0.0"
+            izz="${1/12*wheel_mass*wheel_radius**2}" />
         </inertial>
     </link>
@@ -165,6 +180,9 @@
         </visual>
         <inertial>
-            <mass value="11.3" />
-             <inertia ixx="0.026" ixy="0.0" ixz="0.0" iyy="0.026" iyz="0.0" izz="0.051"/>
+            <mass value="${wheel_mass}" />
+            <inertia ixx="${1/12*wheel_mass*(3*wheel_radius**2+wheel_width)}"
+            ixy="0.0" ixz="0.0"
+            iyy="${1/12*wheel_mass*(3*wheel_radius**2+wheel_width)}"  iyz="0.0"
+            izz="${1/12*wheel_mass*wheel_radius**2}" />
         </inertial>
     </link>

Commit message: yop

File: ackerman_robot/urdf/ackermann.urdf.xacro (robot description, xacro)
@@ -232,28 +232,30 @@
         </ros2_control>
     </xacro:unless>
-  <xacro:if value="$(arg sim_mode)">
-    <ros2_control name="GazeboSystem" type="system">
-        <hardware>
-        <plugin>gz_ros2_control/GazeboSimSystem</plugin>
-        </hardware>
-        <joint name="rear_left_wheel_joint">
-        <command_interface name="velocity" />
-        <state_interface name="velocity" />
-        <state_interface name="position" />
-        </joint>
-        <joint name="rear_right_wheel_joint">
-        <command_interface name="velocity" />
-        <state_interface name="velocity" />
-        <state_interface name="position" />
-        </joint>
-        <joint name="left_wheel_steering_joint">
-        <command_interface name="position" />
-        <state_interface name="position" />
-        </joint>
-        <joint name="right_wheel_steering_joint">
-        <command_interface name="position" />
-        <state_interface name="position" />
-        </joint>
-    </ros2_control>
+    <xacro:if value="$(arg sim_mode)">
+        <ros2_control name="GazeboSystem" type="system">
+            <hardware>
+            <plugin>gz_ros2_control/GazeboSimSystem</plugin>
+            </hardware>
+            <joint name="rear_left_wheel_joint">
+                <command_interface name="velocity" />
+                <state_interface name="velocity" />
+                <state_interface name="position" />
+            </joint>
+            <joint name="rear_right_wheel_joint">
+                <command_interface name="velocity" />
+                <state_interface name="velocity" />
+                <state_interface name="position" />
+            </joint>
+                <joint name="left_wheel_steering_joint">
+                <command_interface name="position" />
+                <state_interface name="position" />
+                <state_interface name="velocity" />
+            </joint>
+            <joint name="right_wheel_steering_joint">
+                <command_interface name="position" />
+                <state_interface name="position" />
+                <state_interface name="velocity" />
+            </joint>
+        </ros2_control>
         <gazebo>
             <plugin filename="gz_ros2_control-system" name="gz_ros2_control::GazeboSimROS2ControlPlugin">
