Commit message: ackermann_robot : added lidar

File: ackerman_robot/urdf/ackermann.urdf.xacro (robot description, xacro)
@@ -25,5 +25,73 @@
     <xacro:property name="wheel_xoff" value="0.12"/>
     <xacro:arg name="sim_mode" default="false"/>
+      <xacro:macro name="inertial_cylinder" params="mass length radius *origin">
+        <inertial>
+            <xacro:insert_block name="origin"/>
+            <mass value="${mass}" />
+            <inertia ixx="${(1/12) * mass * (3*radius*radius + length*length)}" ixy="0.0" ixz="0.0"
+                    iyy="${(1/12) * mass * (3*radius*radius + length*length)}" iyz="0.0"
+                    izz="${(1/2) * mass * (radius*radius)}" />
+        </inertial>
+    </xacro:macro>
     <link name="base_link" />
+   <!-- <joint name="base_footprint_joint" type="fixed">
+        <parent link="base_link"/>
+        <child link="base_footprint"/>
+        <origin xyz="0 0 0" rpy="0 0 0"/>
+    </joint>
+     <link name="base_footprint">
+    </link>-->
+    <!-- LIDAR   -->
+     <joint name="laser_joint" type="fixed">
+        <parent link="chassis"/>
+        <child link="laser_frame"/>
+        <origin xyz="0.022 0 0.095" rpy="0 0 0"/>
+    </joint>
+    <link name="laser_frame">
+        <visual>
+            <geometry>
+                <cylinder radius="0.02" length="0.02"/>
+            </geometry>
+            <material name="Orange"/>
+        </visual>
+        <visual>
+            <origin xyz="0 0 -0.02"/>
+            <geometry>
+                <cylinder radius="0.01" length="0.1"/>
+            </geometry>
+            <material name="Black"/>
+        </visual>
+        <collision>
+            <geometry>
+                <cylinder radius="0.02" length="0.02"/>
+            </geometry>
+        </collision>
+        <xacro:inertial_cylinder mass="0.1" length="0.02" radius="0.02">
+            <origin xyz="0 0 0" rpy="0 0 0"/>
+        </xacro:inertial_cylinder>
+    </link>
+    <gazebo reference="laser_frame">
+        <material>Gazebo/Red</material>
+        <sensor name="laser" type="gpu_lidar">
+            <pose> 0 0 0 0 0 0 </pose>
+            <visualize>false</visualize>
+            <update_rate>10</update_rate>
+            <lidar>
+                <scan>
+                    <horizontal>
+                        <samples>360</samples>
+                        <min_angle>-3.14</min_angle>
+                        <max_angle>3.14</max_angle>
+                    </horizontal>
+                </scan>
+                <range>
+                    <min>0.3</min>
+                    <max>12</max>
+                </range>
+            </lidar>
+           <topic>scan</topic>
+            <gz_frame_id>laser_frame</gz_frame_id>
+        </sensor>
+    </gazebo>
     <!-- Chassis -->
     <link name="chassis">
@@ -69,7 +137,8 @@
         <inertial>
            <mass value="${base_mass}" />
-           <inertia ixx="${1/12 * base_mass * (base_height**2 + base_length ** 2)}" ixy="0.0" ixz="0.0"
-            iyy="${1/12 * base_mass * (base_height ** 2 + base_width ** 2)}" iyz="0.0"
-            izz="${1/12 * base_mass * (base_width ** 2 + base_length ** 2)}" />
+           <inertia ixx="${1/12*wheel_mass*(3*wheel_radius**2+wheel_width)}"
+            ixy="0.0" ixz="0.0"
+            iyy="${1/12*wheel_mass*(3*wheel_radius**2+wheel_width)}"  iyz="0.0"
+            izz="${1/12*wheel_mass*wheel_radius**2}" />
         </inertial>
     </link>
@@ -79,5 +148,5 @@
         <child link="rear_left_wheel" />
         <axis xyz="0 0 1" />
-        <dynamics damping="0.2" />
+        <dynamics damping="0.02" />
     </joint>
     <!-- rear right wheel Link -->
@@ -107,5 +176,5 @@
         <child link="rear_right_wheel" />
         <axis xyz="0 0 1" />
-        <dynamics damping="0.2" />
+        <dynamics damping="0.02" />
     </joint>
     <link name="left_wheel_steering">
@@ -120,5 +189,5 @@
         <child link="left_wheel_steering" />
         <axis xyz="0 1 0" />
-        <dynamics damping="0.2" />
+        <dynamics damping="0.02" />
         <limit effort="10000.0" lower="-0.57" upper="0.57" velocity="30"/>
     </joint>
@@ -137,5 +206,5 @@
         <child link="right_wheel_steering" />
         <axis xyz="0 1 0" />
-        <dynamics damping="0.2" />
+        <dynamics damping="0.02" />
         <limit effort="10000.0" lower="-0.57" upper="0.57" velocity="30"/>
     </joint>
@@ -165,5 +234,5 @@
         <child link="front_left_wheel" />
         <axis xyz="0 0 1" />
-        <dynamics damping="0.2" />
+        <dynamics damping="0.02" />
     </joint>
     <link name="front_right_wheel">
@@ -192,5 +261,5 @@
         <child link="front_right_wheel" />
         <axis xyz="0 0 1" />
-        <dynamics damping="0.2" />
+        <dynamics damping="0.02" />
     </joint>
     <xacro:unless value="$(arg sim_mode)">

Commit message: ackerman_robot: slam

File: ackerman_robot/urdf/ackermann.urdf.xacro (robot description, xacro)
@@ -35,5 +35,5 @@
     </xacro:macro>
     <link name="base_link" />
-   <!-- <joint name="base_footprint_joint" type="fixed">
+    <joint name="base_footprint_joint" type="fixed">
         <parent link="base_link"/>
         <child link="base_footprint"/>
@@ -41,5 +41,5 @@
     </joint>
      <link name="base_footprint">
-    </link>-->
+    </link>
     <!-- LIDAR   -->
      <joint name="laser_joint" type="fixed">
@@ -135,11 +135,7 @@
             <material name="Black" />
         </visual>
-        <inertial>
-           <mass value="${base_mass}" />
-           <inertia ixx="${1/12*wheel_mass*(3*wheel_radius**2+wheel_width)}"
-            ixy="0.0" ixz="0.0"
-            iyy="${1/12*wheel_mass*(3*wheel_radius**2+wheel_width)}"  iyz="0.0"
-            izz="${1/12*wheel_mass*wheel_radius**2}" />
-        </inertial>
+        <xacro:inertial_cylinder mass="${wheel_mass}" length="${wheel_width}" radius="${wheel_radius}">
+            <origin xyz="0 0 0" rpy="0 0 0"/>
+        </xacro:inertial_cylinder>
     </link>
     <joint name="rear_left_wheel_joint" type="continuous">
@@ -163,11 +159,7 @@
             <material name="Black" />
         </visual>
-        <inertial>
-            <mass value="${wheel_mass}" />
-            <inertia ixx="${1/12*wheel_mass*(3*wheel_radius**2+wheel_width)}"
-            ixy="0.0" ixz="0.0"
-            iyy="${1/12*wheel_mass*(3*wheel_radius**2+wheel_width)}"  iyz="0.0"
-            izz="${1/12*wheel_mass*wheel_radius**2}" />
-        </inertial>
+        <xacro:inertial_cylinder mass="${wheel_mass}" length="${wheel_width}" radius="${wheel_radius}">
+            <origin xyz="0 0 0" rpy="0 0 0"/>
+        </xacro:inertial_cylinder>
     </link>
     <joint name="rear_right_wheel_joint" type="continuous">
@@ -221,11 +213,7 @@
             <material name="Black" />
         </visual>
-        <inertial>
-            <mass value="${wheel_mass}" />
-            <inertia ixx="${1/12*wheel_mass*(3*wheel_radius**2+wheel_width)}"
-            ixy="0.0" ixz="0.0"
-            iyy="${1/12*wheel_mass*(3*wheel_radius**2+wheel_width)}"  iyz="0.0"
-            izz="${1/12*wheel_mass*wheel_radius**2}" />
-        </inertial>
+        <xacro:inertial_cylinder mass="${wheel_mass}" length="${wheel_width}" radius="${wheel_radius}">
+            <origin xyz="0 0 0" rpy="0 0 0"/>
+        </xacro:inertial_cylinder>
     </link>
     <joint name="front_left_wheel_joint" type="continuous">
@@ -248,11 +236,7 @@
             <material name="Black" />
         </visual>
-        <inertial>
-            <mass value="${wheel_mass}" />
-            <inertia ixx="${1/12*wheel_mass*(3*wheel_radius**2+wheel_width)}"
-            ixy="0.0" ixz="0.0"
-            iyy="${1/12*wheel_mass*(3*wheel_radius**2+wheel_width)}"  iyz="0.0"
-            izz="${1/12*wheel_mass*wheel_radius**2}" />
-        </inertial>
+        <xacro:inertial_cylinder mass="${wheel_mass}" length="${wheel_width}" radius="${wheel_radius}">
+            <origin xyz="0 0 0" rpy="0 0 0"/>
+        </xacro:inertial_cylinder>
     </link>
     <joint name="front_right_wheel_joint" type="continuous">
